File: reform-wifi.kicad_pcb (KiCad board)
At the start: 4 copper layers, 30 x 51 mm, 24 parts, among them J1 Conn_01x20, J2 Bus_PCI_Express_Mini, J3 Bus_M.2_Socket_E, X1 ECS-327MVATX-2-CN-TR3

Commit message: reannotate schematic
Parts:
- moved D1 0.25 mm to (89.0, 60.5)
- moved R7 0.25 mm to (92.0, 60.5)
- renumbered J3 to J2, J2 to J3, R2 to R1, R1 to R10, R3 to R2, R4 to R3, R5 to R4, R7 to R5, R8 to R6, R9 to R7, R10 to R8, R6 to R9, TP3 to TP1, TP1 to TP2, TP5 to TP3, TP2 to TP5
Routing:
- net PCIE3_RX_P: track 41.8 -> 40.1 mm
- net PCIE3_RX_N: track 41.8 -> 40.0 mm
