File: reform-wifi.kicad_pcb (KiCad board)
At the start: 4 copper layers, 30 x 50.8 mm, 24 parts, among them J1 Conn_01x20, J2 Bus_M.2_Socket_E, J3 Bus_PCI_Express_Mini, X1 ECS-327MVATX-2-CN-TR3

Commit message: update for revision 1
Parts:
- added C1: 100n, Capacitor_SMD:C_0603_1608Metric, F.Cu at (111.0, 35.6)
- added C2: 100n, Capacitor_SMD:C_0603_1608Metric, F.Cu at (89.5, 22.1)
- C3: renamed from C1; value 0.1uF -> 100n
- moved X1 3.93 mm to (111.0, 29.0)
- moved C3 3.81 mm to (111.0, 31.5)
- moved R10 3.81 mm to (111.0, 33.0), turned to 180 degrees
- moved R3 2.78 mm to (111.2, 24.4)
- moved R1 1.92 mm to (111.0, 40.1)
- moved R2 1.92 mm to (111.0, 41.6)
- moved R5 1.92 mm to (111.0, 37.1)
- moved R6 1.92 mm to (111.0, 38.6)
- moved TP1 1.20 mm to (104.2, 36.3)
- moved TP2 1.20 mm to (104.2, 34.1)
- moved TP3 1.00 mm to (98.3, 38.5)
- moved TP4 1.00 mm to (98.3, 36.3)
- moved TP5 1.00 mm to (98.3, 34.1)
- moved R4 0.90 mm to (111.2, 22.9)
- moved R9 0.30 mm to (92.7, 22.1)
Connections:
- J1 pad 10: PCIE3_TX_N -> RK_UART1_RTS_1V8
- J1 pad 11: PCIE3_TX_P -> RK_UART1_CTS_1V8
- J1 pad 12: GND -> RK_UART1_TX_1V8
- J1 pad 13: PCIE3_RX_N -> RK_UART1_RX_1V8
- J1 pad 14: PCIE3_RX_P -> RK_WIFI_GPIO1
- J1 pad 15: GND -> RK_WIFI_GPIO2
- J1 pad 16: PCIE3_CLK_N -> GND
- J1 pad 17: PCIE3_CLK_P -> USB_P
- J1 pad 18: GND -> USB_N
- J1 pad 19: +5V -> unconnected-(J1-Pin_19-Pad19)
- J1 pad 2: USB_P -> SDIO_CLK
- J1 pad 20: +5V -> unconnected-(J1-Pin_20-Pad20)
- J1 pad 3: USB_N -> GND
- J1 pad 4: GND -> SDIO_CMD
- J1 pad 5: RK_WIFI_GPIO0 -> SDIO_D0
- J1 pad 6: RK_WIFI_GPIO1 -> SDIO_D1
- J1 pad 7: RK_WIFI_GPIO2 -> SDIO_D2
- J1 pad 8: RK_WIFI_GPIO3 -> SDIO_D3
- J2 pad 11: SDIO_CMD -> unconnected-(J2-SDIO_CMD-Pad11)
- J2 pad 13: SDIO_D0 -> unconnected-(J2-SDIO_DATA0-Pad13)
- J2 pad 15: SDIO_D1 -> unconnected-(J2-SDIO_DATA1-Pad15)
- J2 pad 17: SDIO_D2 -> unconnected-(J2-SDIO_DATA2-Pad17)
- J2 pad 19: SDIO_D3 -> unconnected-(J2-SDIO_DATA3-Pad19)
- J2 pad 22: RK_UART1_TX_1V8 -> unconnected-(J2-UART_RXD-Pad22)
- J2 pad 32: RK_UART1_RX_1V8 -> unconnected-(J2-UART_TXD-Pad32)
- J2 pad 34: RK_UART1_RTS_1V8 -> unconnected-(J2-UART_CTS-Pad34)
- J2 pad 36: RK_UART1_CTS_1V8 -> unconnected-(J2-UART_RTS-Pad36)
- J2 pad 52: RK_WIFI_GPIO0 -> PERST
- J2 pad 53: RK_WIFI_GPIO1 -> CLKREQ
- J2 pad 55: RK_WIFI_GPIO2 -> WAKE
- J2 pad 9: SDIO_CLK -> unconnected-(J2-SDIO_CLK-Pad9)
- J3 pad 1: unconnected-(J3-~{WAKE}-Pad1) -> WAKE
- J3 pad 11: unconnected-(J3-REFCLK--Pad11) -> PCIE3_CLK_N
- J3 pad 13: unconnected-(J3-REFCLK+-Pad13) -> PCIE3_CLK_P
- J3 pad 20: unconnected-(J3-~{W_DISABLE}-Pad20) -> W_DISABLE
- J3 pad 22: unconnected-(J3-~{PERST}-Pad22) -> PERST
- J3 pad 23: unconnected-(J3-PERn0-Pad23) -> PCIE3_RX_N
- J3 pad 25: unconnected-(J3-PERp0-Pad25) -> PCIE3_RX_P
- J3 pad 31: unconnected-(J3-PETn0-Pad31) -> PCIE3_TX_N
- J3 pad 33: unconnected-(J3-PETp0-Pad33) -> PCIE3_TX_P
- J3 pad 7: unconnected-(J3-~{CLKREQ}-Pad7) -> CLKREQ
- R1 pad 2: RK_WIFI_GPIO0 -> PERST
- R2 pad 1: RK_WIFI_GPIO0 -> PERST
- R3 pad 1: RK_WIFI_GPIO1 -> CLKREQ
- R4 pad 1: RK_WIFI_GPIO2 -> WAKE
- R5 pad 1: RK_WIFI_GPIO3 -> W_DISABLE
Routing:
- net +3V3: track 144.3 -> 90.2 mm, vias 5 -> 12
- net RK_WIFI_GPIO1: track 47.9 -> 0.00 mm, vias 2 -> 0
- net RK_WIFI_GPIO2: track 44.0 -> 0.00 mm, vias 2 -> 0
- net PCIE3_TX_N: track 47.9 -> 6.08 mm
- net PCIE3_TX_P: track 47.8 -> 6.08 mm
- net PCIE3_RX_P: track 40.1 -> 6.66 mm, vias 2 -> 0
- net PCIE3_RX_N: track 40.0 -> 6.66 mm, vias 2 -> 0
- net RK_WIFI_GPIO0: track 32.2 -> 0.00 mm, vias 2 -> 0
- net PERST: track 0.00 -> 30.0 mm, vias 0 -> 1
- net PCIE3_CLK_N: track 41.7 -> 12.9 mm
- net PCIE3_CLK_P: track 41.7 -> 12.9 mm
- net W_DISABLE: track 0.00 -> 22.7 mm, vias 0 -> 1
- net RK_WIFI_GPIO3: track 19.9 -> 0.00 mm, vias 2 -> 0
- net CLKREQ: track 0.00 -> 19.7 mm, vias 0 -> 2
- net WAKE: track 0.00 -> 19.2 mm
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- added copper zone on B.Cu, net +3V3
- added copper zone on F.Cu, net +3V3
Other:
- board text added: "for revision 1 2026-02-23"
