File: reform-wifi.kicad_sch (KiCad schematic)
At the start: 23 parts, among them J1 Conn_01x20, J2 Bus_PCI_Express_Mini, J3 Bus_M.2_Socket_E, X1 ECS-327MVATX-2-CN-TR3

Commit message: reannotate schematic
Parts:
- H1: LCSC C2916321 -> C2916320
- J2: renamed from J3; LCSC C41447443 -> C5163551
- J3: renamed from J2; now not fitted
- renumbered R2 to R1, R1 to R10, R3 to R2, R4 to R3, R5 to R4, R7 to R5, R8 to R6, R9 to R7, R10 to R8, R6 to R9, TP3 to TP1, TP1 to TP2, TP5 to TP3, TP2 to TP5
Changed lines of the file:
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@@
 		(dnp no)
 		(fields_autoplaced yes)
-		(property "Reference" "J3"
+		(property "Reference" "J2"
 			(at 201.5333 40.64 0)
 			(effects
@@
 			)
 		)
-		(property "LCSC" "C41447443"
+		(property "LCSC" "C5163551"
 			(at 199.39 91.44 0)
 			(effects
@@
 			(project ""
 				(path "/a96e4190-6a37-435c-99bf-69421967be4e"
-					(reference "J3")
+					(reference "J2")
 					(unit 1)
 				)
@@
 		(in_bom yes)
 		(on_board yes)
-		(dnp no)
+		(dnp yes)
 		(fields_autoplaced yes)
-		(property "Reference" "J2"
+		(property "Reference" "J3"
 			(at 56.7533 162.56 0)
 			(effects
@@
 			(project ""
 				(path "/a96e4190-6a37-435c-99bf-69421967be4e"
-					(reference "J2")
+					(reference "J3")
 					(unit 1)
 				)
@@
 		(dnp yes)
 		(fields_autoplaced yes)
-		(property "Reference" "R2"
+		(property "Reference" "R1"
 			(at 107.95 35.5599 0)
 			(effects
@@
 			(project "nref-wifi-m2"
 				(path "/a96e4190-6a37-435c-99bf-69421967be4e"
-					(reference "R2")
+					(reference "R1")
 					(unit 1)
 				)
@@
 		(dnp no)
 		(fields_autoplaced yes)
-		(property "Reference" "R7"
+		(property "Reference" "R5"
 			(at 254 64.7699 0)
 			(effects
@@
 			(project "nref-wifi-m2"
 				(path "/a96e4190-6a37-435c-99bf-69421967be4e"
-					(reference "R7")
+					(reference "R5")
 					(unit 1)
 				)
@@
 		(dnp no)
 		(fields_autoplaced yes)
-		(property "Reference" "#PWR01"
+		(property "Reference" "#PWR08"
 			(at 46.99 97.79 0)
 			(effects
@@
 			(project ""
 				(path "/a96e4190-6a37-435c-99bf-69421967be4e"
-					(reference "#PWR01")
+					(reference "#PWR08")
 					(unit 1)
 				)
@@
 		(dnp no)
 		(fields_autoplaced yes)
-		(property "Reference" "R9"
+		(property "Reference" "R7"
 			(at 264.16 96.5199 0)
 			(effects
@@
 			(project "nref-wifi-m2"
 				(path "/a96e4190-6a37-435c-99bf-69421967be4e"
-					(reference "R9")
+					(reference "R7")
 					(unit 1)
 				)
@@
 		(dnp no)
 		(fields_autoplaced yes)
-		(property "Reference" "#PWR010"
+		(property "Reference" "#PWR012"
 			(at 157.48 163.83 0)
 			(effects
@@
 			(project ""
 				(path "/a96e4190-6a37-435c-99bf-69421967be4e"
-					(reference "#PWR010")
+					(reference "#PWR012")
 					(unit 1)
 				)
@@
 		(dnp no)
 		(fields_autoplaced yes)
-		(property "Reference" "R8"
+		(property "Reference" "R6"
 			(at 264.16 64.7699 0)
 			(effects
@@
 			(project ""
 				(path "/a96e4190-6a37-435c-99bf-69421967be4e"
-					(reference "R8")
+					(reference "R6")
 					(unit 1)
 				)
@@
 		(dnp yes)
 		(fields_autoplaced yes)
-		(property "Reference" "R6"
+		(property "Reference" "R9"
 			(at 149.86 110.4899 0)
 			(effects
@@
 			(project "nref-wifi-m2"
 				(path "/a96e4190-6a37-435c-99bf-69421967be4e"
-					(reference "R6")
+					(reference "R9")
 					(unit 1)
 				)
@@
 		(dnp no)
 		(fields_autoplaced yes)
-		(property "Reference" "R1"
+		(property "Reference" "R10"
 			(at 99.06 153.6699 0)
 			(effects
@@
 			(project "nref-wifi-m2"
 				(path "/a96e4190-6a37-435c-99bf-69421967be4e"
-					(reference "R1")
+					(reference "R10")
 					(unit 1)
 				)
@@
 		(dnp no)
 		(fields_autoplaced yes)
-		(property "Reference" "#PWR02"
+		(property "Reference" "#PWR013"
 			(at 52.07 172.72 0)
 			(effects
@@
 			(project ""
 				(path "/a96e4190-6a37-435c-99bf-69421967be4e"
-					(reference "#PWR02")
+					(reference "#PWR013")
 					(unit 1)
 				)
@@
 		(on_board yes)
 		(dnp no)
-		(property "Reference" "#PWR011"
+		(property "Reference" "#PWR03"
 			(at 199.39 34.29 0)
 			(effects
@@
 			(project "nref-wifi-m2"
 				(path "/a96e4190-6a37-435c-99bf-69421967be4e"
-					(reference "#PWR011")
+					(reference "#PWR03")
 					(unit 1)
 				)
@@
 		(on_board yes)
 		(dnp no)
-		(property "Reference" "#PWR08"
+		(property "Reference" "#PWR05"
 			(at 105.41 71.12 0)
 			(effects
@@
 			(project "nref-wifi-m2"
 				(path "/a96e4190-6a37-435c-99bf-69421967be4e"
-					(reference "#PWR08")
+					(reference "#PWR05")
 					(unit 1)
 				)
@@
 			)
 		)
-		(property "LCSC" "C2916321"
+		(property "LCSC" "C2916320"
 			(at 157.48 154.94 0)
 			(effects
@@
 		(on_board yes)
 		(dnp no)
-		(property "Reference" "#PWR07"
+		(property "Reference" "#PWR02"
 			(at 105.41 34.29 0)
 			(effects
@@
 			(project "nref-wifi-m2"
 				(path "/a96e4190-6a37-435c-99bf-69421967be4e"
-					(reference "#PWR07")
+					(reference "#PWR02")
 					(unit 1)
 				)
@@
 		(on_board yes)
 		(dnp no)
-		(property "Reference" "#PWR05"
+		(property "Reference" "#PWR011"
 			(at 101.6 153.67 0)
 			(effects
@@
 			(project "nref-wifi-m2"
 				(path "/a96e4190-6a37-435c-99bf-69421967be4e"
-					(reference "#PWR05")
+					(reference "#PWR011")
 					(unit 1)
 				)
@@
 		(dnp no)
 		(fields_autoplaced yes)
-		(property "Reference" "R10"
+		(property "Reference" "R8"
 			(at 279.4 96.5199 0)
 			(effects
@@
 			(project "nref-wifi-m2"
 				(path "/a96e4190-6a37-435c-99bf-69421967be4e"
-					(reference "R10")
+					(reference "R8")
 					(unit 1)
 				)
@@
 		(on_board yes)
 		(dnp no)
-		(property "Reference" "#PWR012"
+		(property "Reference" "#PWR010"
 			(at 199.39 149.86 0)
 			(effects
@@
 			(project "nref-wifi-m2"
 				(path "/a96e4190-6a37-435c-99bf-69421967be4e"
-					(reference "#PWR012")
+					(reference "#PWR010")
 					(unit 1)
 				)
@@
 		(dnp yes)
 		(fields_autoplaced yes)
-		(property "Reference" "TP3"
+		(property "Reference" "TP1"
 			(at 240.03 62.2299 90)
 			(effects
@@
 			(project "nref-wifi-m2"
 				(path "/a96e4190-6a37-435c-99bf-69421967be4e"
-					(reference "TP3")
+					(reference "TP1")
 					(unit 1)
 				)
@@
 		(dnp no)
 		(fields_autoplaced yes)
-		(property "Reference" "R3"
+		(property "Reference" "R2"
 			(at 107.95 57.1499 0)
 			(effects
@@
 			(project "nref-wifi-m2"
 				(path "/a96e4190-6a37-435c-99bf-69421967be4e"
-					(reference "R3")
+					(reference "R2")
 					(unit 1)
 				)
@@
 		(on_board yes)
 		(dnp no)
-		(property "Reference" "#PWR013"
+		(property "Reference" "#PWR04"
 			(at 261.62 63.5 0)
 			(effects
@@
 			(project "nref-wifi-m2"
 				(path "/a96e4190-6a37-435c-99bf-69421967be4e"
-					(reference "#PWR013")
+					(reference "#PWR04")
 					(unit 1)
 				)
@@
 		(on_board yes)
 		(dnp no)
-		(property "Reference" "#PWR03"
+		(property "Reference" "#PWR01"
 			(at 71.12 30.48 0)
 			(effects
@@
 			(project "nref-wifi-m2"
 				(path "/a96e4190-6a37-435c-99bf-69421967be4e"
-					(reference "#PWR03")
+					(reference "#PWR01")
 					(unit 1)
 				)
@@
 		(dnp no)
 		(fields_autoplaced yes)
-		(property "Reference" "R5"
+		(property "Reference" "R4"
 			(at 123.19 57.1499 0)
 			(effects
@@
 			(project "nref-wifi-m2"
 				(path "/a96e4190-6a37-435c-99bf-69421967be4e"
-					(reference "R5")
+					(reference "R4")
 					(unit 1)
 				)
@@
 		(dnp yes)
 		(fields_autoplaced yes)
-		(property "Reference" "TP1"
+		(property "Reference" "TP2"
 			(at 232.41 64.7699 90)
 			(effects
@@
 			(project "nref-wifi-m2"
 				(path "/a96e4190-6a37-435c-99bf-69421967be4e"
-					(reference "TP1")
+					(reference "TP2")
 					(unit 1)
 				)
@@
 		(dnp yes)
 		(fields_autoplaced yes)
-		(property "Reference" "TP5"
+		(property "Reference" "TP3"
 			(at 265.43 123.1899 90)
 			(effects
@@
 			(project "nref-wifi-m2"
 				(path "/a96e4190-6a37-435c-99bf-69421967be4e"
-					(reference "TP5")
+					(reference "TP3")
 					(unit 1)
 				)
@@
 		(on_board yes)
 		(dnp no)
-		(property "Reference" "#PWR014"
+		(property "Reference" "#PWR06"
 			(at 261.62 93.98 0)
 			(effects
@@
 			(project "nref-wifi-m2"
 				(path "/a96e4190-6a37-435c-99bf-69421967be4e"
-					(reference "#PWR014")
+					(reference "#PWR06")
 					(unit 1)
 				)
@@
 		(dnp no)
 		(fields_autoplaced yes)
-		(property "Reference" "#PWR06"
+		(property "Reference" "#PWR014"
 			(at 101.6 195.58 0)
 			(effects
@@
 			(project "nref-wifi-m2"
 				(path "/a96e4190-6a37-435c-99bf-69421967be4e"
-					(reference "#PWR06")
+					(reference "#PWR014")
 					(unit 1)
 				)
@@
 		(on_board yes)
 		(dnp no)
-		(property "Reference" "#PWR04"
+		(property "Reference" "#PWR07"
 			(at 71.12 99.06 0)
 			(effects
@@
 			(project "nref-wifi-m2"
 				(path "/a96e4190-6a37-435c-99bf-69421967be4e"
-					(reference "#PWR04")
+					(reference "#PWR07")
 					(unit 1)
 				)
@@
 		(dnp yes)
 		(fields_autoplaced yes)
-		(property "Reference" "TP2"
+		(property "Reference" "TP5"
 			(at 236.22 128.2699 90)
 			(effects
@@
 			(project ""
 				(path "/a96e4190-6a37-435c-99bf-69421967be4e"
-					(reference "TP2")
+					(reference "TP5")
 					(unit 1)
 				)
@@
 		(dnp no)
 		(fields_autoplaced yes)
-		(property "Reference" "R4"
+		(property "Reference" "R3"
 			(at 115.57 57.1499 0)
 			(effects
@@
 			(project "nref-wifi-m2"
 				(path "/a96e4190-6a37-435c-99bf-69421967be4e"
-					(reference "R4")
+					(reference "R3")
 					(unit 1)
 				)

Commit message: update for revision 1
Parts:
- added C1, C2: 100n, Capacitor_SMD:C_0603_1608Metric, symbol Device:C_Small
- C3: renamed from C1; value 0.1uF -> 100n
- J3: now fitted
Connections:
- net +3V3: now also C1.1, C2.1
- net GND: now also J1.16 (Pin_16), J1.3 (Pin_3), C1.2, C2.2; no longer J1.12 (Pin_12), J1.15 (Pin_15), J1.18 (Pin_18), J1.4 (Pin_4)
- net PCIE3_CLK_N: now also J3.11 (REFCLK-); no longer J1.16 (Pin_16)
- net PCIE3_CLK_P: now also J3.13 (REFCLK+); no longer J1.17 (Pin_17)
- net PCIE3_RX_N: now also J3.23 (PERn0); no longer J1.13 (Pin_13)
- net PCIE3_RX_P: now also J3.25 (PERp0); no longer J1.14 (Pin_14)
- net PCIE3_TX_N: now also J3.31 (PETn0); no longer J1.10 (Pin_10)
- net PCIE3_TX_P: now also J3.33 (PETp0); no longer J1.11 (Pin_11)
- net RK_UART1_CTS_1V8: now also J1.11 (Pin_11); no longer J2.36 (UART_RTS)
- net RK_UART1_RTS_1V8: now also J1.10 (Pin_10); no longer J2.34 (UART_CTS)
- net RK_UART1_RX_1V8: now also J1.13 (Pin_13); no longer J2.32 (UART_TXD)
- net RK_UART1_TX_1V8: now also J1.12 (Pin_12); no longer J2.22 (UART_RXD)
- net RK_WIFI_GPIO1: now also J1.14 (Pin_14); no longer J1.6 (Pin_6), J2.53 (~{CLKREQ0}), R3.1
- net RK_WIFI_GPIO2: now also J1.15 (Pin_15); no longer J1.7 (Pin_7), J2.55 (~{PEWAKE0}), R4.1
- net SDIO_CLK: now also J1.2 (Pin_2); no longer J2.9 (SDIO_CLK)
- net SDIO_CMD: now also J1.4 (Pin_4); no longer J2.11 (SDIO_CMD)
- net SDIO_D0: now also J1.5 (Pin_5); no longer J2.13 (SDIO_DATA0)
- net SDIO_D1: now also J1.6 (Pin_6); no longer J2.15 (SDIO_DATA1)
- net SDIO_D2: now also J1.7 (Pin_7); no longer J2.17 (SDIO_DATA2)
- net SDIO_D3: now also J1.8 (Pin_8); no longer J2.19 (SDIO_DATA3)
- net USB_N: now also J1.18 (Pin_18); no longer J1.3 (Pin_3)
- net USB_P: now also J1.17 (Pin_17); no longer J1.2 (Pin_2)
- net WAKE: now reaches J3.1 (~{WAKE})
- net WAKE: now also J2.55 (~{PEWAKE0}), R4.1
- net W_DISABLE: now reaches J3.20 (~{W_DISABLE})
- net W_DISABLE: now also R5.1
- net PERST: now reaches J3.22 (~{PERST})
- net PERST: now also J2.52 (~{PERST0}), R1.2, R2.1
- net CLKREQ: now reaches J3.7 (~{CLKREQ})
- net CLKREQ: now also J2.53 (~{CLKREQ0}), R3.1
- net +5V: no longer names the net of J1.19 (Pin_19)
- net +5V: no longer J1.20 (Pin_20)
- removed net RK_WIFI_GPIO0: J1.5 (Pin_5), J2.52 (~{PERST0}), R1.2, R2.1
- removed net RK_WIFI_GPIO3: J1.8 (Pin_8), R5.1
- no-connect marks 63 -> 67
Other:
- note added: "3.3V or 5V from RCORE"
- note added: "WiFi/BT/Internal Expansion Revision 1 RCORE boards only"
- note removed: "3V3 levels"
- note removed: "Attn: N/P"
- note removed: "CLKREQ_N"
- note removed: "DET_WAKE"
- note removed: "NC"
- note removed: "PWR_EN"
- note removed: "RST_B"
- note removed: "WiFi/BT/Internal Expansion (flipped! need same side contacts cable!)"
- moved on the sheet: D1, D2, R7, R8
